File: tinyCore-hat.kicad_pcb (KiCad board)
At the start: 4 copper layers, 48.3 x 48.3 mm, 3 parts, among them J2 PPTC081LFBN-RC, J3 PPTC081LFBN-RC, J4 HTSW-109-07-X-SJ

Commit message: fix(pcb): board outline
Other:
- board size 48.3 x 48.3 mm -> 49 x 48.8 mm
Changed lines of the file:
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@@
 		)
 	)
-	(gr_line
-		(start 158.501105 129.145735)
-		(end 138.501105 129.145735)
+	(gr_poly
+		(pts
+			(xy 158.5 81) (xy 173 95.003595) (xy 173 116) (xy 158.501105 129.5) (xy 138.25 129.25) (xy 124 115)
+			(xy 124.5 94.25) (xy 138.75 80.75)
+		)
 		(stroke
 			(width 0.05)
 			(type solid)
 		)
+		(fill no)
 		(layer "Edge.Cuts")
 	)
 	(gr_line
-		(start 124.358965 115.003595)
-		(end 124.358965 95.003595)
-		(stroke
-			(width 0.05)
-			(type solid)
-		)
-		(layer "Edge.Cuts")
-	)
-	(gr_line
-		(start 138.501105 129.145735)
-		(end 124.358965 115.003595)
-		(stroke
-			(width 0.05)
-			(type solid)
-		)
-		(layer "Edge.Cuts")
-	)
-	(gr_line
-		(start 172.643235 95.003595)
-		(end 172.643235 115.003595)
-		(stroke
-			(width 0.05)
-			(type solid)
-		)
-		(layer "Edge.Cuts")
-	)
-	(gr_line
-		(start 124.358965 95.003595)
-		(end 138.501105 80.861465)
-		(stroke
-			(width 0.05)
-			(type solid)
-		)
-		(layer "Edge.Cuts")
-	)
-	(gr_line
-		(start 158.501105 80.861465)
-		(end 172.643235 95.003595)
-		(stroke
-			(width 0.05)
-			(type solid)
-		)
-		(layer "Edge.Cuts")
-	)
-	(gr_line
-		(start 172.643235 115.003595)
-		(end 158.501105 129.145735)
-		(stroke
-			(width 0.05)
-			(type solid)
-		)
-		(layer "Edge.Cuts")
-	)
-	(gr_line
-		(start 138.501105 129.145735)
-		(end 158.501105 129.145735)
+		(start 138.25 129.25)
+		(end 158.501105 129.5)
 		(stroke
 			(width 0.0127)
@@
 		(polygon
 			(pts
-				(xy 124.359995 129.137245) (xy 124.359995 80.861465) (xy 172.643235 80.861465) (xy 172.643235 129.137245)
+				(xy 173 95) (xy 173 116) (xy 158.5 129.5) (xy 138.25 129.25) (xy 124 115) (xy 124.5 94.5) (xy 138.5 80.861465)
+				(xy 158.5 81)
 			)
 		)
@@
 		(polygon
 			(pts
-				(xy 124.359995 129.137245) (xy 124.359995 80.861465) (xy 172.643235 80.861465) (xy 172.643235 129.137245)
-			)
-		)
+				(xy 173 95) (xy 173 116) (xy 158.5 129.5) (xy 138.25 129.25) (xy 124 115) (xy 124.5 94.25) (xy 138.75 80.75)
+				(xy 158.5 81)
+			)
+		)

Commit message: fix(pcb): board outline
Other:
- board size 49 x 48.8 mm -> 49 x 47.5 mm
Changed lines of the file:
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@@
 	(gr_poly
 		(pts
-			(xy 158.5 81) (xy 173 95.003595) (xy 173 116) (xy 158.501105 129.5) (xy 138.25 129.25) (xy 124 115)
-			(xy 124.5 94.25) (xy 138.75 80.75)
+			(xy 158.5 81) (xy 173 95.003595) (xy 173 116) (xy 160.75 128.25) (xy 136.75 128) (xy 124 116) (xy 124.25 94.25)
+			(xy 138.75 80.75)
 		)
 		(stroke
